File: pcb/JayPad.kicad_pcb (KiCad board)
At the start: 2 copper layers, 113 x 70.8 mm, 65 parts, among them M1 MOUDLE-SEEEDUINO-XIAO, SW1 PEC11-4215F-S24

Commit message: Added one lil cat decor
Parts:
- added G***: LOGO, LOGO, B.Cu at (102.0, 81.5)
- added G***: LOGO, LOGO, B.Cu at (186.2, 124.8)
Other:
- board text added: "Made with by Jayx2u"
- board text removed: "Created by Jayx2u"
